File: pcb/Braille-Display-with-Inductor-Solenoids/Braille-Display-with-Inductor-Solenoids.kicad_pcb (KiCad board)
At the start: 2 copper layers, 90 x 93 mm, 106 parts, among them J1 Screw_Terminal_01x02, J2 Screw_Terminal_01x02, J4 Conn_01x03, J5 Conn_01x02, J6 Conn_01x08, J7 Screw_Terminal_01x02, J8 Barrel_Jack_Switch, U1 RP2040-Zero, U103 INA219AxD, U2 EG27324, U26 74HC595, U27 74HC595, U3 EG27324, U4 EG27324, U5 EG27324, U6 EG27324, U7 EG27324, U8 EG27324, U9 EG27324

Commit message: pcb: WIP - High power and repeated routing
Parts:
- removed J4: Conn_01x03, Connector_PinHeader_2.54mm:PinHeader_1x03_P2.54mm_Vertical
- moved R120 150.3 mm to (57.5, 110.0)
- moved R116 147.4 mm to (57.5, 98.5)
- moved R108 141.5 mm to (57.8, 37.0)
- moved S14 141.1 mm to (57.2, 115.0), turned to 90 degrees
- moved R112 140.9 mm to (57.8, 47.5)
- moved S13 139.7 mm to (57.2, 103.5), turned to 90 degrees
- moved S4 136.1 mm to (57.2, 32.0), turned to 90 degrees
- moved S8 135.6 mm to (57.2, 42.2), turned to 90 degrees
- moved R109 129.1 mm to (63.8, 37.0)
- moved R113 126.8 mm to (63.8, 47.5)
- moved S5 125.7 mm to (63.2, 32.0), turned to 90 degrees
- moved R121 124.6 mm to (63.5, 110.0)
- moved S9 124.3 mm to (63.2, 42.2), turned to 90 degrees
- moved R117 123.2 mm to (63.5, 98.5)
- moved S16 116.7 mm to (63.2, 115.0), turned to 90 degrees
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Connections:
- U1 pad 7: Net-(J4-Pin_1) -> unconnected-(U1-GP26-Pad7)_1
- U1 pad 8: Net-(J4-Pin_2) -> I2C_SCL
- U1 pad 9: Net-(J4-Pin_3) -> I2C_SDA
Routing:
- net VDC: track 0.00 -> 189.5 mm, vias 0 -> 13
- net GND: track 0.00 -> 151.3 mm, vias 0 -> 14
- net +3V3: track 0.00 -> 141.5 mm
- net Net-(J7-Pin_1): track 0.00 -> 36.2 mm
- net /Braille_Cells_and_Controls/Braille_Cell3/MAG_BOTTOM_A: track 0.00 -> 20.3 mm, vias 0 -> 2
- net /Braille_Cells_and_Controls/Braille_Cell2/MAG_BOTTOM_A: track 0.00 -> 20.3 mm, vias 0 -> 2
- net /Braille_Cells_and_Controls/Braille_Cell/MAG_BOTTOM_A: track 0.00 -> 20.3 mm, vias 0 -> 2
- net /Braille_Cells_and_Controls/Braille_Cell1/MAG_BOTTOM_A: track 0.00 -> 20.3 mm, vias 0 -> 2
- net /Braille_Cells_and_Controls/Braille_Cell2/MAG_TOP_A: track 0.00 -> 19.6 mm, vias 0 -> 2
- net /Braille_Cells_and_Controls/Braille_Cell3/MAG_TOP_A: track 0.00 -> 19.6 mm, vias 0 -> 2
- net /Braille_Cells_and_Controls/Braille_Cell1/MAG_TOP_A: track 0.00 -> 19.6 mm, vias 0 -> 2
- net /Braille_Cells_and_Controls/Braille_Cell/MAG_TOP_A: track 0.00 -> 19.6 mm, vias 0 -> 2
- net /Braille_Cells_and_Controls/Braille_Cell3/MAG_BOTTOM_SW_B: track 0.00 -> 18.1 mm
- net /Braille_Cells_and_Controls/Braille_Cell2/MAG_BOTTOM_SW_B: track 0.00 -> 18.1 mm
- net /Braille_Cells_and_Controls/Braille_Cell1/MAG_BOTTOM_SW_B: track 0.00 -> 18.1 mm
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